Commit message: Frame corrected

File: urdf/vero_model.urdf (robot description, URDF)
Before this commit: robot myfirst, 4 links, 3 joints
Joints:
- joint base_to_camera: origin xyz=1 0 0.1 rpy=0 0 -1.5708 -> xyz=0.15 0 0.1 rpy=0 0 -1.5708
- joint base_to_lidar1: origin xyz=1 1 0.1 rpy=0 0 0.7853 -> xyz=0.15 0.15 0.1 rpy=0 0 0.7853
- joint base_to_lidar2: origin xyz=-1 -1 0.1 rpy=0 0 -2.356194 -> xyz=-0.15 -0.15 0.1 rpy=0 0 -2.356194
