Commit message: Tuned for CONA

File: urdf/pioneer.urdf (robot description, URDF)
Before this commit: robot Pioneer_2-AT_8, 12 links, 11 joints
Links:
- removed link cam_link
- added link astra_link; visual box size=0.02 0.04 0.02
Joints:
- removed joint actuator_cam_joint
- added joint actuator_astra_joint: type continuous, parent cam_actuator_link, child astra_link, origin xyz=0 0 0.03 rpy=0 0 0, axis 0 0 1
